Commit message: navigation ready, slam works, odom is smooth

File: src/base101/base101_control/urdf/base101.hardware.xacro (robot description, xacro)
@@ -7,46 +7,11 @@
   <xacro:arg name="simulator" default="none"/>
   <xacro:include filename="$(find base101_description)/urdf/base101.xacro"/>
-  <!-- =================================================================
-       Hardware ros2_control block — Axon 2 firmware bridge.
-       The on-board Axon 2 firmware (axon-firmware) runs the DDSM210 wheel
-       drivers and exposes them as a ROS 2 node over zenoh: it subscribes to
-       /motor_manager/base_cmd (a Float64MultiArray of per-wheel velocities in
-       rad/s) and publishes /motor_manager/joint_states. base101_control_plugin
-       bridges the diff_drive_controller's per-wheel velocity command/state
-       interfaces to those topics.
-       IMPORTANT: the wheel <joint> order below is the order the bridge packs
-       into base_cmd[]. It must match the firmware's command_index in
-       axon-firmware/src/ros/axon_config.h: [0]=FL [1]=FR [2]=BL [3]=BR.
-       The joint NAMES must match the firmware's joint_states names
-       (front_left_wheel_joint, ...) so the state round-trip lines up.
-       Run the host zenoh router + rmw_zenoh first — see HARDWARE.md.
-       ================================================================= -->
-  <ros2_control name="base101_hw_system" type="system">
-    <hardware>
-      <plugin>base101_control_plugin/ROS2ControlBridge</plugin>
-      <param name="base_cmd_topic">/motor_manager/base_cmd</param>
-      <param name="state_topic">/motor_manager/joint_states</param>
-      <param name="publish_if_unchanged">true</param>
-    </hardware>
-    <joint name="front_left_wheel_joint">
-      <command_interface name="velocity"/>
-      <state_interface name="position"/>
-      <state_interface name="velocity"/>
-    </joint>
-    <joint name="front_right_wheel_joint">
-      <command_interface name="velocity"/>
-      <state_interface name="position"/>
-      <state_interface name="velocity"/>
-    </joint>
-    <joint name="back_left_wheel_joint">
-      <command_interface name="velocity"/>
-      <state_interface name="position"/>
-      <state_interface name="velocity"/>
-    </joint>
-    <joint name="back_right_wheel_joint">
-      <command_interface name="velocity"/>
-      <state_interface name="position"/>
-      <state_interface name="velocity"/>
-    </joint>
-  </ros2_control>
+  <!-- No <ros2_control> block here: the Axon 2 firmware (base101-fw) owns
+       locomotion — /link101/cmd_vel in — but odometry is NOT fused on the
+       firmware: it only exposes raw wheel odometry (/link101/odom/raw) and
+       raw IMU (/link101/imu), no TF of its own. A host-side EKF
+       (base101_bringup_hw/launch/robot.launch.py) fuses those into /odom +
+       odom -> base_link instead. No /joint_states either way (the wheel
+       joints just sit at 0 in RViz — cosmetic only, nothing downstream needs
+       them). See HARDWARE.md for the full topic contract. -->
 </robot>

File: src/base101/base101_description/urdf/chassis.xacro (robot description, xacro)
@@ -676,5 +676,11 @@
      height of the optical window between the base and the spinning cap
      (CAD z = 14.5 mm, i.e. 96.5 mm off the floor). /scan is stamped in
-     it and slam/nav consume it from there. -->
+     it and slam/nav consume it from there.
+     lidar_mount_1/lidar_1 are zero-rotation relative to their parents (real
+     CAD placement, taken verbatim from the export) but lidar_frame_joint
+     below carries an extra yaw=pi: confirmed (2026-09-21) that raw /scan's
+     angle=0 is the physical rear of the robot, not lidar_1's own +X the
+     CAD export otherwise assumes — a frame-definition mismatch, not the
+     physical mounting or the driver. See that joint's comment. -->
 <link name="lidar_mount_1">
   <inertial>
@@ -729,5 +735,12 @@
 <link name="lidar_frame"/>
 <joint name="lidar_frame_joint" type="fixed">
-  <origin xyz="-0.021498 -0.0215 0.030313" rpy="0 0 0"/>
+  <!-- yaw=pi, confirmed (2026-09-21): raw /scan's angle=0 is the physical
+       rear, not lidar_1's own +X as the zero here originally assumed — see
+       the lidar section's header comment above. Only this joint carries the
+       correction (not lidar_mount_joint/lidar_joint above), since those two
+       are real CAD placement for the mount bracket/sensor body meshes and
+       are correct as exported; this one is purely the scan-origin frame TF
+       consumers (SLAM, costmaps) read /scan through. -->
+  <origin xyz="-0.021498 -0.0215 0.030313" rpy="0 0 3.141593"/>
   <parent link="lidar_1"/>
   <child link="lidar_frame"/>

Commit message: mojuco

File: src/base101/base101_control/urdf/base101.hardware.xacro (robot description, xacro)
@@ -7,46 +7,8 @@
   <xacro:arg name="simulator" default="none"/>
   <xacro:include filename="$(find base101_description)/urdf/base101.xacro"/>
-  <!-- =================================================================
-       Hardware ros2_control block — Axon 2 firmware bridge.
-       The on-board Axon 2 firmware (axon-firmware) runs the DDSM210 wheel
-       drivers and exposes them as a ROS 2 node over zenoh: it subscribes to
-       /motor_manager/base_cmd (a Float64MultiArray of per-wheel velocities in
-       rad/s) and publishes /motor_manager/joint_states. base101_control_plugin
-       bridges the diff_drive_controller's per-wheel velocity command/state
-       interfaces to those topics.
-       IMPORTANT: the wheel <joint> order below is the order the bridge packs
-       into base_cmd[]. It must match the firmware's command_index in
-       axon-firmware/src/ros/axon_config.h: [0]=FL [1]=FR [2]=BL [3]=BR.
-       The joint NAMES must match the firmware's joint_states names
-       (front_left_wheel_joint, ...) so the state round-trip lines up.
-       Run the host zenoh router + rmw_zenoh first — see HARDWARE.md.
-       ================================================================= -->
-  <ros2_control name="base101_hw_system" type="system">
-    <hardware>
-      <plugin>base101_control_plugin/ROS2ControlBridge</plugin>
-      <param name="base_cmd_topic">/motor_manager/base_cmd</param>
-      <param name="state_topic">/motor_manager/joint_states</param>
-      <param name="publish_if_unchanged">true</param>
-    </hardware>
-    <joint name="front_left_wheel_joint">
-      <command_interface name="velocity"/>
-      <state_interface name="position"/>
-      <state_interface name="velocity"/>
-    </joint>
-    <joint name="front_right_wheel_joint">
-      <command_interface name="velocity"/>
-      <state_interface name="position"/>
-      <state_interface name="velocity"/>
-    </joint>
-    <joint name="back_left_wheel_joint">
-      <command_interface name="velocity"/>
-      <state_interface name="position"/>
-      <state_interface name="velocity"/>
-    </joint>
-    <joint name="back_right_wheel_joint">
-      <command_interface name="velocity"/>
-      <state_interface name="position"/>
-      <state_interface name="velocity"/>
-    </joint>
-  </ros2_control>
+  <!-- No <ros2_control> block: locomotion bypasses ros2_control entirely on
+       real hardware. The Axon 2 firmware owns the DDSM210 wheel drivers and
+       talks ROS topics directly over zenoh — it subscribes to /cmd_vel and
+       publishes /odom — so there is no per-wheel command/state interface for
+       a SystemInterface to bridge. See HARDWARE.md. -->
 </robot>

File: src/base101/base101_description/urdf/base101.xacro (robot description, xacro)
@@ -53,5 +53,7 @@
   </xacro:if>
   <!-- simulator=isaac: driven natively from base101_isaac (no ros2_control).
-       simulator=none: real-hw ros2_control comes from base101_control's
-       hardware xacro (base101.hardware.xacro). -->
+       simulator=none: real hardware — no ros2_control block at all. The
+       Axon 2 firmware owns locomotion directly over zenoh (/cmd_vel in,
+       /odom out); base101.hardware.xacro just wraps this with
+       simulator:=none forced. -->
 </robot>
